Commit message: Update URDF and add MJCF data structure

File: mujoco_ros2_control_demos/demo_resources/car/urdf/car.urdf (robot description, URDF)
Before this commit: robot car, 6 links, 5 joints
Links:
- link chassis: geometry collision box size=0.12 0.15 0.055; visual mesh filename=package://mujoco_ros2_control_demos/demo_resources/car/mesh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 scale=1 1 1
- link wheel: geometry collision cylinder length=0.015 radius=0.025; visual mesh filename=package://mujoco_ros2_control_demos/demo_resources/car/mesh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 scale=1 1 1
- link wheel_1: geometry collision cylinder length=0.015 radius=0.025; visual mesh filename=package://mujoco_ros2_control_demos/demo_resources/car/mesh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 scale=1 1 1
- link wheel_2: geometry collision cylinder length=0.015 radius=0.025; visual mesh filename=package://mujoco_ros2_control_demos/demo_resources/car/mesh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 scale=1 1 1
- link wheel_3: geometry collision cylinder length=0.015 radius=0.025; visual mesh filename=package://mujoco_ros2_control_demos/demo_resources/car/mesh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 scale=1 1 1
